File: MAM_GND_V5.brd (EAGLE design)
At the start: 53.4 x 86.4 mm, 4 parts, among them X1 SMA-142-0701-801/806

Commit message: Add files via upload
Routing:
- added copper zone on layer 1, net GND
Other:
- board size 53.4 x 86.4 mm -> 53.4 x 87.6 mm
Changed lines of the file:
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@@
 <drawing>
 <settings>
-<setting alwaysvectorfont="no"/>
+<setting alwaysvectorfont="yes"/>
 <setting verticaltext="up"/>
 </settings>
@@
 <board>
 <plain>
-<wire x1="9.525" y1="0" x2="62.8775" y2="0.005" width="0" layer="20"/>
-<wire x1="62.8775" y1="0.005" x2="62.8525" y2="86.355" width="0" layer="20"/>
+<wire x1="9.525" y1="-1.27" x2="62.8775" y2="-1.265" width="0" layer="20"/>
+<wire x1="62.8775" y1="-1.265" x2="62.8525" y2="86.355" width="0" layer="20"/>
 <wire x1="62.8525" y1="86.355" x2="9.525" y2="86.35" width="0" layer="20"/>
-<wire x1="9.525" y1="86.35" x2="9.525" y2="0" width="0" layer="20"/>
+<wire x1="9.525" y1="86.35" x2="9.525" y2="-1.27" width="0" layer="20"/>
 </plain>
 <attributes>
@@
 <contactref element="JP1" pad="10"/>
 <contactref element="U$2" pad="P$1"/>
+<polygon width="0.508" layer="1">
+<vertex x="17.145" y="86.36"/>
+<vertex x="55.245" y="86.36"/>
+<vertex x="62.865" y="78.74"/>
+<vertex x="62.865" y="6.35"/>
+<vertex x="55.245" y="-1.27"/>
+<vertex x="17.145" y="-1.27"/>
+<vertex x="9.525" y="6.35"/>
+<vertex x="9.525" y="78.74"/>
+</polygon>
 <wire x1="51.4096" y1="83.7946" x2="51.4096" y2="83.7946" width="0" layer="19" extent="1-16"/>
 <wire x1="42.5704" y1="83.7946" x2="51.4096" y2="83.7946" width="0" layer="19" extent="1-1"/>
 <wire x1="42.5704" y1="83.7946" x2="42.5704" y2="83.7946" width="0" layer="19" extent="1-16"/>
 <wire x1="16.51" y1="54.61" x2="42.5704" y2="83.7946" width="0" layer="19" extent="1-1"/>
-<wire x1="57.785" y1="28.575" x2="51.4096" y2="83.7946" width="0" layer="19" extent="1-1"/>
-<wire x1="57.785" y1="26.035" x2="57.785" y2="28.575" width="0" layer="19" extent="1-1"/>
-<wire x1="39.36" y1="15.885" x2="57.785" y2="26.035" width="0" layer="19" extent="1-1"/>
+<wire x1="39.36" y1="15.885" x2="16.51" y2="54.61" width="0" layer="19" extent="1-1"/>
+<wire x1="57.785" y1="26.035" x2="39.36" y2="15.885" width="0" layer="19" extent="1-1"/>
+<wire x1="57.785" y1="28.575" x2="57.785" y2="26.035" width="0" layer="19" extent="1-1"/>
 </signal>
 <signal name="MOSI">
